Commit message: commit

File: ros_ur_driver/install/ur_description/share/ur_description/urdf/ur5_robotiq85_gripper.urdf.xacro (robot description, xacro)
@@ -1,9 +1,8 @@
 <?xml version="1.0"?>
-<robot name="ur5" xmlns:xacro="http://www.ros.org/wiki/xacro">
+<robot xmlns:xacro="http://www.ros.org/wiki/xacro" name="ur5_2f" >
   <xacro:include filename="$(find ur_description)/urdf/ur.urdf.xacro" />
   <xacro:include filename="$(find robotiq_description)/urdf/robotiq_85_gripper.urdf.xacro" />
+  <!-- parameters -->
   <!-- Robotiq Coupler -->
-  <!--  + Height added by the coupler: 8mm -->
-  <!--  + Reference frame: at the middle (4mm) -->
   <link name="robotiq_coupler">
     <visual>
@@ -62,6 +61,6 @@
     <gripper name="gazebo_gripper">
       <grasp_check>
-        <attach_steps>2</attach_steps>    <!-- default: 20 -->
-        <detach_steps>2</detach_steps>    <!-- default: 40 -->
+        <attach_steps>2</attach_steps>
+        <detach_steps>2</detach_steps>
         <min_contact_count>3</min_contact_count>
       </grasp_check>

File: ros_ur_driver/src/install/ur_description/share/ur_description/urdf/ur5_robotiq85_gripper.urdf.xacro (robot description, xacro)
@@ -1,5 +1,20 @@
 <?xml version="1.0"?>
-<robot name="ur5" xmlns:xacro="http://www.ros.org/wiki/xacro">
+<robot xmlns:xacro="http://www.ros.org/wiki/xacro" name="ur5" >
   <xacro:include filename="$(find ur_description)/urdf/ur.urdf.xacro" />
+<!-- parameters -->
+   <xacro:arg name="prefix" default="" />
+   <xacro:arg name="joint_limit_params" default=""/>
+   <xacro:arg name="kinematics_params" default=""/>
+   <xacro:arg name="physical_params" default=""/>
+   <xacro:arg name="visual_params" default=""/>
+   <xacro:arg name="transmission_hw_interface" default=""/>
+   <xacro:arg name="safety_limits" default="false"/>
+   <xacro:arg name="safety_pos_margin" default="0.15"/>
+   <xacro:arg name="safety_k_position" default="20"/>
+   <!-- ros2_control related parameters -->
+   <xacro:arg name="use_fake_hardware" default="false" />
+   <xacro:arg name="fake_sensor_commands" default="false" />
+   <!-- initial position -->
+   <xacro:arg name="initial_positions_file" default="$(find ur_description)/config/initial_positions.yaml"/>
   <xacro:include filename="$(find robotiq_description)/urdf/robotiq_85_gripper.urdf.xacro" />
   <!-- Robotiq Coupler -->
@@ -27,5 +42,5 @@
   <joint name="robotiq_coupler_joint" type="fixed">
     <origin xyz="0 0 0.004" rpy="0 0 ${-pi/2.0}" />
-    <parent link="tool0"/>
+    <parent link="flange"/>
     <child link="robotiq_coupler"/>
   </joint>
@@ -47,5 +62,5 @@
   </xacro:robotiq_85_gripper>
   <!-- Gazebo FT sensor plugin -->
-  <gazebo reference="wrist_3_joint">
+  <!-- <gazebo reference="wrist_3_joint">
     <provideFeedback>true</provideFeedback>
   </gazebo>
@@ -57,11 +72,11 @@
       <jointName>wrist_3_joint</jointName>
     </plugin>
-  </gazebo>
+  </gazebo> -->
   <!-- Gazebo grasping plugin -->
-  <gazebo>
+  <!-- <gazebo>
     <gripper name="gazebo_gripper">
       <grasp_check>
-        <attach_steps>2</attach_steps>    <!-- default: 20 -->
-        <detach_steps>2</detach_steps>    <!-- default: 40 -->
+        <attach_steps>2</attach_steps>
+        <detach_steps>2</detach_steps>
         <min_contact_count>3</min_contact_count>
       </grasp_check>
@@ -70,4 +85,4 @@
       <palm_link>robotiq_85_base_link</palm_link>
     </gripper>
-  </gazebo>
+  </gazebo> -->
 </robot>

File: ros_ur_driver/src/install/ur_description/share/ur_description/urdf/ur_macro.xacro (robot description, xacro)
@@ -50,5 +50,5 @@
     physical_parameters_file
     visual_parameters_file
-    transmission_hw_interface:=hardware_interface/EffortJointInterface
+    transmission_hw_interface:=hardware_interface/PositionJointInterface
     safety_limits:=false
     safety_pos_margin:=0.15

File: ros_ur_driver/src/install/ur_description/share/ur_description/urdf/ur_macro_right.xacro (robot description, xacro)
@@ -50,5 +50,5 @@
     physical_parameters_file
     visual_parameters_file
-    transmission_hw_interface:=hardware_interface/EffortJointInterface
+    transmission_hw_interface:=hardware_interface/PositionJointInterface
     safety_limits:=false
     safety_pos_margin:=0.15
