Commit message: debugging

File: ros_ur_driver/install/ur_description/share/ur_description/urdf/ur.ros2_control.xacro (robot description, xacro)
@@ -7,5 +7,5 @@
     input_recipe_filename tf_prefix
     hash_kinematics robot_ip
-    robot_ip reverse_port:=50001 script_sender_port:=50002 trajectory_port:=50003">
+    reverse_port:=50001 script_sender_port:=50002 trajectory_port:=50003">
     <ros2_control name="${name}" type="system">
       <hardware>

File: ros_ur_driver/install/ur_description/share/ur_description/urdf/ur.urdf.xacro (robot description, xacro)
@@ -15,4 +15,7 @@
    <xacro:arg name="safety_pos_margin" default="0.15"/>
    <xacro:arg name="safety_k_position" default="20"/>
+   <xacro:arg name="reverse_port" default="50001"/>
+   <xacro:arg name="script_sender_port" default="50002"/>
+   <xacro:arg name="trajectory_port" default="50003"/>
    <!-- ros2_control related parameters -->
    <xacro:arg name="use_fake_hardware" default="false" />
@@ -34,4 +37,8 @@
      use_fake_hardware="$(arg use_fake_hardware)"
      fake_sensor_commands="$(arg fake_sensor_commands)"
-     initial_positions="${load_yaml(initial_positions_file)}" />
+     initial_positions="${load_yaml(initial_positions_file)}"
+     reverse_port="$(arg reverse_port)"
+     script_sender_port="$(arg script_sender_port)"
+     trajectory_port="$(arg trajectory_port)"
+     />
 </robot>

File: ros_ur_driver/install/ur_description/share/ur_description/urdf/ur5_robotiq85_gripper.urdf.xacro (robot description, xacro)
@@ -3,5 +3,4 @@
   <xacro:include filename="$(find ur_description)/urdf/ur.urdf.xacro" />
   <xacro:include filename="$(find robotiq_description)/urdf/robotiq_85_gripper.urdf.xacro" />
-  <!-- parameters -->
   <!-- Robotiq Coupler -->
   <link name="robotiq_coupler">
@@ -34,11 +33,4 @@
     <material>Gazebo/FlatBlack</material>
   </gazebo>
-  <!-- Equivalent to the OpenRAVE manipulator denso_robotiq_85_gripper -->
-  <!-- <link name="denso_robotiq_85_gripper" /> -->
-  <!-- <joint name="manipulator_dummy_joint" type="fixed"> -->
-  <!--   <origin xyz="0 0 0.1441" rpy="0 0 0" /> -->
-  <!--   <parent link="robotiq_coupler"/> -->
-  <!--   <child link="denso_robotiq_85_gripper"/> -->
-  <!-- </joint> -->
   <!-- Attach the robotiq 85 gripper -->
   <xacro:robotiq_85_gripper prefix="" parent="robotiq_coupler" >

File: ros_ur_driver/install/ur_description/share/ur_description/urdf/ur_macro.xacro (robot description, xacro)
@@ -56,5 +56,6 @@
     use_fake_hardware:=false
     fake_sensor_commands:=false
-    initial_positions:=${dict(shoulder_pan_joint=0.0,shoulder_lift_joint=-1.57,elbow_joint=0.0,wrist_1_joint=-1.57,wrist_2_joint=0.0,wrist_3_joint=0.0)}">
+    initial_positions:=${dict(shoulder_pan_joint=0.0,shoulder_lift_joint=-1.57,elbow_joint=0.0,wrist_1_joint=-1.57,wrist_2_joint=0.0,wrist_3_joint=0.0)}
+    reverse_port script_sender_port trajectory_port">
     <!-- Load configuration data from the provided .yaml files -->
     <xacro:read_model_data
@@ -81,5 +82,9 @@
       tf_prefix=""
       hash_kinematics="${kinematics_hash}"
-      robot_ip="$(arg robot_ip)" />
+      robot_ip="$(arg robot_ip)"
+      reverse_port="$(arg reverse_port)"
+      script_sender_port="$(arg script_sender_port)"
+      trajectory_port="$(arg trajectory_port)"
+    />
     <!-- Add URDF transmission elements (for ros_control) -->
     <!--<xacro:ur_arm_transmission prefix="${prefix}" hw_interface="${transmission_hw_interface}" />-->

File: ros_ur_driver/src/robotiq/robotiq_description/urdf/robotiq_85_gripper.urdf.xacro (robot description, xacro)
@@ -27,17 +27,17 @@
       </inertial>
     </link>
-    <joint name="${prefix}robotiq_85_left_knuckle_joint" type="revolute">
+    <joint name="${prefix}robotiq_85_left_knuckle_joint" type="fixed"> <!-- revolute -->
       <parent link="${prefix}robotiq_85_base_link"/>
       <child link="${prefix}robotiq_85_left_knuckle_link"/>
       <axis xyz="0 0 1"/>
       <origin rpy="${pi} 0.0 0.0" xyz="0.05490451627 0.03060114443 0.0"/>
-      <limit lower="0.0" upper="0.80285" velocity="0.5" effort="1000"/>
-    </joint>
-    <joint name="${prefix}robotiq_85_right_knuckle_joint" type="continuous">
+      <!-- <limit lower="0.0" upper="0.80285" velocity="0.5" effort="1000"/> -->
+    </joint>
+    <joint name="${prefix}robotiq_85_right_knuckle_joint" type="fixed"> <!-- continuous-->
       <parent link="${prefix}robotiq_85_base_link"/>
       <child link="${prefix}robotiq_85_right_knuckle_link"/>
       <axis xyz="0 0 1"/>
       <origin rpy="0.0 0.0 0.0" xyz="0.05490451627 -0.03060114443 0.0"/>
-      <limit lower="-3.14" upper="3.14" velocity="100.0" effort="1000"/>
+      <!-- <limit lower="-3.14" upper="3.14" velocity="100.0" effort="1000"/> -->
       <mimic joint="${prefix}robotiq_85_left_knuckle_joint"/>
     </joint>
@@ -128,5 +128,5 @@
       </inertial>
     </link>
-    <joint name="${prefix}robotiq_85_left_inner_knuckle_joint" type="continuous">
+    <joint name="${prefix}robotiq_85_left_inner_knuckle_joint" type="fixed"> <!-- continuous -->
       <parent link="${prefix}robotiq_85_base_link"/>
       <child link="${prefix}robotiq_85_left_inner_knuckle_link"/>
@@ -136,5 +136,5 @@
       <mimic joint="${prefix}robotiq_85_left_knuckle_joint" offset="0"/>
     </joint>
-    <joint name="${prefix}robotiq_85_right_inner_knuckle_joint" type="continuous">
+    <joint name="${prefix}robotiq_85_right_inner_knuckle_joint" type="fixed"> <!-- continuous-->
       <parent link="${prefix}robotiq_85_base_link"/>
       <child link="${prefix}robotiq_85_right_inner_knuckle_link"/>
@@ -182,5 +182,5 @@
       </inertial>
     </link>
-    <joint name="${prefix}robotiq_85_left_finger_tip_joint" type="continuous">
+    <joint name="${prefix}robotiq_85_left_finger_tip_joint" type="continuous"> <!-- continuous-->
       <parent link="${prefix}robotiq_85_left_inner_knuckle_link"/>
       <child link="${prefix}robotiq_85_left_finger_tip_link"/>
@@ -190,5 +190,5 @@
       <mimic joint="${prefix}robotiq_85_left_knuckle_joint" multiplier="-1"/>
     </joint>
-    <joint name="${prefix}robotiq_85_right_finger_tip_joint" type="continuous">
+    <joint name="${prefix}robotiq_85_right_finger_tip_joint" type="continuous"> <!-- continuous-->
       <parent link="${prefix}robotiq_85_right_inner_knuckle_link"/>
       <child link="${prefix}robotiq_85_right_finger_tip_link"/>
